File: mcu.kicad_sch (KiCad schematic)
At the start: 49 parts, among them J1 STM32_TRACE, J15 EXPANSION_1, J2 STM32 SWD, Q1 2N7002, Q2 2N7002, Q3 2N7002, Q4 2N7002, Q5 2N7002, Q6 2N7002, SW1 RESET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

Commit message: fix uart gps
Parts:
- removed J2: STM32 SWD, Connector_PinHeader_1.27mm:PinHeader_2x05_P1.27mm_Vertical_SMD, symbol Connector:Conn_ARM_JTAG_SWD_10
- added R47: 4k7, symbol Device:R
Connections:
- net +3V3: now also R47.1
- net GPS.RX: now also U1.119 (PD5); no longer U1.122 (PD6)
- net GPS.TX: now also U1.122 (PD6); no longer U1.119 (PD5)
- net OCTOSPI_NCS: now also R47.2
- no-connect marks 7 -> 6
